Commit message: moveitでロボットアーム動かせた

File: Lerobot_ros2/src/so101_follower_description/urdf/so101_follower.urdf.xacro (robot description, xacro)
@@ -3,5 +3,9 @@
 <!-- Onshape https://cad.onshape.com/documents/7715cc284bb430fe6dab4ffd/w/4fd0791b683777b02f8d975a/e/826c553ede3b7592eb9ca800 -->
 <robot name="so101_follower" xmlns:xacro="http://www.ros.org/wiki/xacro">
-  <xacro:include filename="$(find so101_hw_interface)/urdf/so101_follower.urdf" />
+  <!-- MoveIt adds its own control block; the legacy hardware launch opts in. -->
+  <xacro:arg name="include_ros2_control" default="false"/>
+  <xacro:if value="$(arg include_ros2_control)">
+    <xacro:include filename="$(find so101_hw_interface)/urdf/so101_follower.urdf"/>
+  </xacro:if>
   <!-- World Link -->
   <link name="world"/>
@@ -319,6 +323,5 @@
     <child link="jaw_link"/>
     <axis xyz="0 0 1"/>
-    <!-- calibrated limits: raw(2047,3489) home(2768) = (-1.110,+1.109) rad -->
-    <limit effort="10" velocity="10" lower="-0.6" upper="1.74533"/>
+    <limit effort="10" velocity="10" lower="-0.222427" upper="0.868233"/>
   </joint>
   <transmission name="gripper_trans">
@@ -338,6 +341,5 @@
     <child link="gripper_link"/>
     <axis xyz="0 0 1"/>
-    <!-- calibrated limits: raw(0,4766) home(2084) = (-3.194,+4.120) rad -->
-    <limit effort="10" velocity="10" lower="-3.194" upper="4.120"/>
+    <limit effort="10" velocity="10" lower="-1.612213" upper="1.612213"/>
   </joint>
   <transmission name="wrist_roll_trans">
@@ -357,6 +359,5 @@
     <child link="wrist_link"/>
     <axis xyz="0 0 1"/>
-    <!-- calibrated limits: raw(588,2917) home(1752) = (-1.786,+1.790) rad -->
-    <limit effort="10" velocity="10" lower="-1.786" upper="1.790"/>
+    <limit effort="10" velocity="10" lower="-1.681242" upper="1.682776"/>
   </joint>
   <transmission name="wrist_flex_trans">
@@ -376,6 +377,5 @@
     <child link="lower_arm_link"/>
     <axis xyz="0 0 1"/>
-    <!-- calibrated limits: raw(976,3130) home(2053) = (-1.653,+1.654) rad -->
-    <limit effort="10" velocity="10" lower="-1.653" upper="1.654"/>
+    <limit effort="10" velocity="10" lower="-1.632155" upper="1.633689"/>
   </joint>
   <transmission name="elbow_flex_trans">
@@ -395,6 +395,5 @@
     <child link="upper_arm_link"/>
     <axis xyz="0 0 1"/>
-    <!-- calibrated limits: raw(740,3370) home(2055) = (-2.018,+2.018) rad -->
-    <limit effort="10" velocity="10" lower="-2.018" upper="2.018"/>
+    <limit effort="10" velocity="10" lower="-1.688912" upper="1.690446"/>
   </joint>
   <transmission name="shoulder_lift_trans">
@@ -414,6 +413,5 @@
     <child link="shoulder_link"/>
     <axis xyz="0 0 1"/>
-    <!-- calibrated limits: raw(745,3424) home(2084) = (-2.055,+2.058) rad -->
-    <limit effort="10" velocity="10" lower="-2.055" upper="2.058"/>
+    <limit effort="10" velocity="10" lower="-1.750272" upper="1.751806"/>
   </joint>
   <transmission name="shoulder_pan_trans">

File: Lerobot_ros2/src/so101_follower_moveit/config/so101_follower.ros2_control.xacro (robot description, xacro)
@@ -1,69 +1,32 @@
 <?xml version="1.0"?>
 <robot xmlns:xacro="http://www.ros.org/wiki/xacro">
-    <xacro:macro name="so101_follower_ros2_control" params="name initial_positions_file:=/dev/null">
-        <ros2_control name="${name}" type="system">
-            <hardware>
-                 <xacro:if value="${initial_positions_file != '/dev/null'}">
-                    <plugin>mock_components/GenericSystem</plugin>
-                 </xacro:if>
-                 <xacro:unless value="${initial_positions_file != '/dev/null'}">
-                    <plugin>topic_based_ros2_control/TopicBasedSystem</plugin>
-                    <param name="joint_commands_topic">/so101_follower/joint_commands</param>
-                    <param name="joint_states_topic">/so101_follower/joint_states</param>
-                 </xacro:unless>
-            </hardware>
-            <joint name="shoulder_pan">
-                <command_interface name="position"/>
-                <state_interface name="position">
-                  <param name="initial_value">${load_yaml(initial_positions_file)['initial_positions']['shoulder_pan'] if initial_positions_file != '/dev/null' else '0.0'}</param>
-                </state_interface>
-                <state_interface name="velocity"/>
-            </joint>
-            <joint name="shoulder_lift">
-                <command_interface name="position"/>
-                <state_interface name="position">
-                    <param name="initial_value">${load_yaml(initial_positions_file)['initial_positions']['shoulder_lift'] if initial_positions_file != '/dev/null' else '0.0'}</param>
-                </state_interface>
-                <state_interface name="velocity"/>
-            </joint>
-            <joint name="elbow_flex">
-                <command_interface name="position"/>
-                <state_interface name="position">
-                    <param name="initial_value">${load_yaml(initial_positions_file)['initial_positions']['elbow_flex'] if initial_positions_file != '/dev/null' else '0.0'}</param>
-                </state_interface>
-                <state_interface name="velocity"/>
-            </joint>
-            <joint name="wrist_flex">
-                <command_interface name="position"/>
-                <state_interface name="position">
-                    <param name="initial_value">${load_yaml(initial_positions_file)['initial_positions']['wrist_flex'] if initial_positions_file != '/dev/null' else '0.0'}</param>
-                </state_interface>
-                <state_interface name="velocity"/>
-            </joint>
-            <joint name="wrist_roll">
-                <command_interface name="position"/>
-                <state_interface name="position">
-                    <param name="initial_value">${load_yaml(initial_positions_file)['initial_positions']['wrist_roll'] if initial_positions_file != '/dev/null' else '0.0'}</param>
-                </state_interface>
-                <state_interface name="velocity"/>
-            </joint>
-            <joint name="wrist_pitch">
-                <command_interface name="position"/>
-                <state_interface name="position"/>
-                <state_interface name="velocity"/>
-            </joint>
-            <joint name="wrist_yaw">
-                <command_interface name="position"/>
-                <state_interface name="position"/>
-                <state_interface name="velocity"/>
-            </joint>
-            <joint name="gripper_jaw">
-                <command_interface name="position"/>
-                <state_interface name="position">
-                    <param name="initial_value">${load_yaml(initial_positions_file)['initial_positions']['gripper'] if initial_positions_file != '/dev/null' else '0.0'}</param>
-                </state_interface>
-                <state_interface name="velocity"/>
-            </joint>
-        </ros2_control>
-    </xacro:macro>
+  <xacro:macro name="so101_follower_ros2_control" params="name use_fake_hardware initial_positions_file">
+    <xacro:property name="initial_positions" value="${xacro.load_yaml(initial_positions_file)['initial_positions']}"/>
+    <ros2_control name="${name}" type="system">
+      <hardware>
+        <xacro:if value="${use_fake_hardware}">
+          <plugin>mock_components/GenericSystem</plugin>
+        </xacro:if>
+        <xacro:unless value="${use_fake_hardware}">
+          <plugin>joint_state_topic_hardware_interface/JointStateTopicSystem</plugin>
+          <param name="joint_commands_topic">/so101_follower/joint_commands</param>
+          <param name="joint_states_topic">/so101_follower/joint_states</param>
+        </xacro:unless>
+      </hardware>
+      <xacro:macro name="controlled_joint" params="joint_name">
+        <joint name="${joint_name}">
+          <command_interface name="position"/>
+          <state_interface name="position">
+            <param name="initial_value">${initial_positions[joint_name]}</param>
+          </state_interface>
+        </joint>
+      </xacro:macro>
+      <xacro:controlled_joint joint_name="shoulder_pan"/>
+      <xacro:controlled_joint joint_name="shoulder_lift"/>
+      <xacro:controlled_joint joint_name="elbow_flex"/>
+      <xacro:controlled_joint joint_name="wrist_flex"/>
+      <xacro:controlled_joint joint_name="wrist_roll"/>
+      <xacro:controlled_joint joint_name="gripper"/>
+    </ros2_control>
+  </xacro:macro>
 </robot>

File: Lerobot_ros2/src/so101_follower_moveit/config/so101_follower.urdf.xacro (robot description, xacro)
@@ -1,15 +1,10 @@
 <?xml version="1.0"?>
 <robot xmlns:xacro="http://www.ros.org/wiki/xacro" name="so101_follower">
-    <xacro:arg name="initial_positions_file" default="initial_positions.yaml" />
-    <xacro:arg name="use_fake_hardware" default="true" />
-    <!-- Import so101_follower urdf file -->
-    <xacro:include filename="$(find so101_follower_description)/urdf/so101_follower.urdf.xacro" />
-    <!-- Import so101_follower ros2_control description -->
-    <xacro:include filename="so101_follower.ros2_control.xacro" />
-    <xacro:if value="$(arg use_fake_hardware)">
-        <xacro:so101_follower_ros2_control name="FakeSystem" initial_positions_file="$(find so101_follower_moveit)/config/initial_positions.yaml"/>
-    </xacro:if>
-    <xacro:unless value="$(arg use_fake_hardware)">
-        <xacro:so101_follower_ros2_control name="so101_follower"/>
-    </xacro:unless>
+  <xacro:arg name="use_fake_hardware" default="true"/>
+  <xacro:arg name="initial_positions_file" default="$(find so101_follower_moveit)/config/initial_positions.yaml"/>
+  <xacro:include filename="$(find so101_follower_description)/urdf/so101_follower.urdf.xacro"/>
+  <xacro:include filename="so101_follower.ros2_control.xacro"/>
+  <xacro:so101_follower_ros2_control name="SO101"
+      use_fake_hardware="$(arg use_fake_hardware)"
+      initial_positions_file="$(arg initial_positions_file)"/>
 </robot>
